File: hardware/S88P.sch (KiCad schematic (older format))
At the start: 79 parts, among them IC1 ATMEGA8-AI, J1 RJ45, J2 RJ45, P1 CONN_3X2, P2 CONN_8, P3 CONN_8

Commit message: Added FTDI Header, decoupled AVREF and added buffer cap on the power line
Parts:
- added C? (x2): 100nF, ~, symbol C
- added C?: 4.7uF, ~, symbol C
- added P4: CONN_6, symbol CONN_6
Connections:
- net GND: now also C?.1, C?.2, P4.1 (GND), P4.2 (CTS)
- net S88OUT: now also P4.4 (TXO)
- net TRACK10: now also IC1.22 (ADC7)
- net TRACK9: now also IC1.19 (ADC6)
- net VCC: now also C?.1, P4.5V (3); no longer IC1.18 (AVCC)
- net at C1.1, IC1.29 (PC6(~RESET~)), P1.5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: now also C?.1
- net at IC1.31 ((TXD)PD1): now also P4.5 (RXI)
- new net: C?.2, IC1.18 (AVCC)
- new net: C?.2, P4.6 (DTR)
- no-connect marks 5 -> 2
