File: hardware/S88P.sch (KiCad schematic (older format))
At the start: 79 parts, among them IC1 ATMEGA8-AI, J1 RJ45, J2 RJ45, P1 CONN_3X2, P2 CONN_8, P3 CONN_8

Commit message: Updates for newer standard schematic symbols
Parts:
- D1: symbol LED -> LED-RESCUE-S88P
Other:
- moved on the sheet: C1, D18, D19, D2, D20, D21, D22, D23, D24, D25, D3, D4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

Commit message: Fixed capacitors and resistor connections
Connections:
- wire segments 234 -> 236
Other:
- moved on the sheet: R15, R16, R17, R18, R19, R20, R21, R22
Changed lines of the file:
@@
 	1050 2350 1050 2500
 Wire Wire Line
-	1050 2250 1600 2250
-Wire Wire Line
 	1050 2100 1050 2250
-Wire Wire Line
-	1600 2150 1050 2150
 Connection ~ 1050 2150
 Text GLabel 1550 2850 0    60   Input ~ 0
@@
 	3500 2250 4700 2250
 Wire Wire Line
-	4700 2350 3500 2350
+	3500 2350 4700 2350
 Wire Wire Line
 	3500 2450 4700 2450
@@
 	6600 1000 6950 1000
 Wire Wire Line
-	6900 1000 6900 1050
+	6900 1000 6900 1100
 $Comp
 L GND #PWR011
@@
 	7750 1500 7750 1450
 Wire Wire Line
-	6900 1450 6900 1500
+	6900 1400 6900 1500
 Connection ~ 6900 1000
 $Comp
@@
 	6600 1700 6950 1700
 Wire Wire Line
-	6900 1700 6900 1750
+	6900 1700 6900 1800
 $Comp
 L GND #PWR013
@@
 	7750 2200 7750 2150
 Wire Wire Line
-	6900 2150 6900 2200
+	6900 2100 6900 2200
 Connection ~ 6900 1700
 $Comp
@@
 	6600 2350 6950 2350
 Wire Wire Line
-	6900 2350 6900 2400
+	6900 2350 6900 2450
 $Comp
 L GND #PWR015
@@
 	7750 2850 7750 2800
 Wire Wire Line
-	6900 2800 6900 2850
+	6900 2750 6900 2850
 Connection ~ 6900 2350
 Connection ~ 7750 2350
@@
 	6600 3050 6950 3050
 Wire Wire Line
-	6900 3050 6900 3100
+	6900 3050 6900 3150
 $Comp
 L GND #PWR017
@@
 	7750 3550 7750 3500
 Wire Wire Line
-	6900 3500 6900 3550
+	6900 3450 6900 3550
 Connection ~ 6900 3050
 Connection ~ 7750 3050
@@
 	6600 3700 6950 3700
 Wire Wire Line
-	6900 3700 6900 3750
+	6900 3700 6900 3800
 $Comp
 L GND #PWR019
@@
 	7750 4200 7750 4150
 Wire Wire Line
-	6900 4150 6900 4200
+	6900 4100 6900 4200
 Connection ~ 6900 3700
 Connection ~ 7750 3700
@@
 	6600 4400 6950 4400
 Wire Wire Line
-	6900 4400 6900 4450
+	6900 4400 6900 4500
 $Comp
 L GND #PWR021
@@
 	7750 4900 7750 4850
 Wire Wire Line
-	6900 4850 6900 4900
+	6900 4800 6900 4900
 Connection ~ 6900 4400
 Connection ~ 7750 4400
@@
 	6600 5050 6950 5050
 Wire Wire Line
-	6900 5050 6900 5100
+	6900 5050 6900 5150
 $Comp
 L GND #PWR023
@@
 	7750 5550 7750 5500
 Wire Wire Line
-	6900 5500 6900 5550
+	6900 5450 6900 5550
 Connection ~ 6900 5050
 Connection ~ 7750 5050
@@
 	6600 5750 6950 5750
 Wire Wire Line
-	6900 5750 6900 5800
+	6900 5750 6900 5850
 $Comp
 L GND #PWR025
@@
 	7750 6250 7750 6200
 Wire Wire Line
-	6900 6200 6900 6250
+	6900 6150 6900 6250
 Connection ~ 6900 5750
 Connection ~ 7750 5750
@@
 L R R15
 U 1 1 50A1F403
-P 9600 1000
-F 0 "R15" V 9680 1000 50  0000 C CNN
-F 1 "1k" V 9600 1000 50  0000 C CNN
-F 2 "" H 9600 1000 60  0001 C CNN
-F 3 "" H 9600 1000 60  0001 C CNN
-	1    9600 1000
+P 9700 1000
+F 0 "R15" V 9780 1000 50  0000 C CNN
+F 1 "1k" V 9700 1000 50  0000 C CNN
+F 2 "" H 9700 1000 60  0001 C CNN
+F 3 "" H 9700 1000 60  0001 C CNN
+	1    9700 1000
 	0    -1   -1   0
 $EndComp
@@
 	10350 1050 10350 1000
 Wire Wire Line
-	9000 1000 9350 1000
-Wire Wire Line
-	9300 1000 9300 1050
+	9000 1000 9550 1000
+Wire Wire Line
+	9300 1000 9300 1100
 $Comp
 L GND #PWR027
@@
 	10350 1500 10350 1450
 Wire Wire Line
-	9300 1450 9300 1500
+	9300 1400 9300 1500
 Connection ~ 9300 1000
 Connection ~ 10350 1000
@@
 L R R16
 U 1 1 50A1F429
-P 9600 1700
-F 0 "R16" V 9680 1700 50  0000 C CNN
-F 1 "1k" V 9600 1700 50  0000 C CNN
-F 2 "" H 9600 1700 60  0001 C CNN
-F 3 "" H 9600 1700 60  0001 C CNN
-	1    9600 1700
+P 9700 1700
+F 0 "R16" V 9780 1700 50  0000 C CNN
+F 1 "1k" V 9700 1700 50  0000 C CNN
+F 2 "" H 9700 1700 60  0001 C CNN
+F 3 "" H 9700 1700 60  0001 C CNN
+	1    9700 1700
 	0    -1   -1   0
 $EndComp
@@
 	10350 1750 10350 1700
 Wire Wire Line
-	9000 1700 9350 1700
-Wire Wire Line
-	9300 1700 9300 1750
+	9000 1700 9550 1700
+Wire Wire Line
+	9300 1700 9300 1800
 $Comp
 L GND #PWR029
@@
 	10350 2200 10350 2150
 Wire Wire Line
-	9300 2150 9300 2200
+	9300 2100 9300 2200
 Connection ~ 9300 1700
 Connection ~ 10350 1700
@@
 L R R17
 U 1 1 50A1F44F
-P 9600 2350
-F 0 "R17" V 9680 2350 50  0000 C CNN
-F 1 "1k" V 9600 2350 50  0000 C CNN
-F 2 "" H 9600 2350 60  0001 C CNN
-F 3 "" H 9600 2350 60  0001 C CNN
-	1    9600 2350
+P 9700 2350
+F 0 "R17" V 9780 2350 50  0000 C CNN
+F 1 "1k" V 9700 2350 50  0000 C CNN
+F 2 "" H 9700 2350 60  0001 C CNN
+F 3 "" H 9700 2350 60  0001 C CNN
+	1    9700 2350
 	0    -1   -1   0
 $EndComp
@@
 	10350 2400 10350 2350
 Wire Wire Line
-	9000 2350 9350 2350
-Wire Wire Line
-	9300 2350 9300 2400
+	9000 2350 9550 2350
+Wire Wire Line
+	9300 2350 9300 2450
 $Comp
 L GND #PWR031
@@
 	10350 2850 10350 2800
 Wire Wire Line
-	9300 2800 9300 2850
+	9300 2750 9300 2850
 Connection ~ 9300 2350
 Connection ~ 10350 2350
@@
 L R R18
 U 1 1 50A1F475
-P 9600 3050
-F 0 "R18" V 9680 3050 50  0000 C CNN
-F 1 "1k" V 9600 3050 50  0000 C CNN
-F 2 "" H 9600 3050 60  0001 C CNN
-F 3 "" H 9600 3050 60  0001 C CNN
-	1    9600 3050
+P 9700 3050
+F 0 "R18" V 9780 3050 50  0000 C CNN
+F 1 "1k" V 9700 3050 50  0000 C CNN
+F 2 "" H 9700 3050 60  0001 C CNN
+F 3 "" H 9700 3050 60  0001 C CNN
+	1    9700 3050
 	0    -1   -1   0
 $EndComp
@@
 	10350 3100 10350 3050
 Wire Wire Line
-	9000 3050 9350 3050
-Wire Wire Line
-	9300 3050 9300 3100
+	9000 3050 9550 3050
+Wire Wire Line
+	9300 3050 9300 3150
 $Comp
 L GND #PWR033
@@
 	10350 3550 10350 3500
 Wire Wire Line
-	9300 3500 9300 3550
+	9300 3450 9300 3550
 Connection ~ 9300 3050
 Connection ~ 10350 3050
@@
 L R R19
 U 1 1 50A1F49B
-P 9600 3700
-F 0 "R19" V 9680 3700 50  0000 C CNN
-F 1 "1k" V 9600 3700 50  0000 C CNN
-F 2 "" H 9600 3700 60  0001 C CNN
-F 3 "" H 9600 3700 60  0001 C CNN
-	1    9600 3700
+P 9700 3700
+F 0 "R19" V 9780 3700 50  0000 C CNN
+F 1 "1k" V 9700 3700 50  0000 C CNN
+F 2 "" H 9700 3700 60  0001 C CNN
+F 3 "" H 9700 3700 60  0001 C CNN
+	1    9700 3700
 	0    -1   -1   0
 $EndComp
@@
 	10350 3750 10350 3700
 Wire Wire Line
-	9000 3700 9350 3700
-Wire Wire Line
-	9300 3700 9300 3750
+	9000 3700 9550 3700
+Wire Wire Line
+	9300 3700 9300 3800
 $Comp
 L GND #PWR035
@@
 	10350 4200 10350 4150
 Wire Wire Line
-	9300 4150 9300 4200
+	9300 4100 9300 4200
 Connection ~ 9300 3700
 Connection ~ 10350 3700
@@
 L R R20
 U 1 1 50A1F4C1
-P 9600 4400
-F 0 "R20" V 9680 4400 50  0000 C CNN
-F 1 "1k" V 9600 4400 50  0000 C CNN
-F 2 "" H 9600 4400 60  0001 C CNN
-F 3 "" H 9600 4400 60  0001 C CNN
-	1    9600 4400
+P 9700 4400
+F 0 "R20" V 9780 4400 50  0000 C CNN
+F 1 "1k" V 9700 4400 50  0000 C CNN
+F 2 "" H 9700 4400 60  0001 C CNN
+F 3 "" H 9700 4400 60  0001 C CNN
+	1    9700 4400
 	0    -1   -1   0
 $EndComp
@@
 	10350 4450 10350 4400
 Wire Wire Line
-	9000 4400 9350 4400
-Wire Wire Line
-	9300 4400 9300 4450
+	9000 4400 9550 4400
+Wire Wire Line
+	9300 4400 9300 4500
 $Comp
 L GND #PWR037
@@
 	10350 4900 10350 4850
 Wire Wire Line
-	9300 4850 9300 4900
+	9300 4800 9300 4900
 Connection ~ 9300 4400
 Connection ~ 10350 4400
@@
 L R R21
 U 1 1 50A1F4E7
-P 9600 5050
-F 0 "R21" V 9680 5050 50  0000 C CNN
-F 1 "1k" V 9600 5050 50  0000 C CNN
-F 2 "" H 9600 5050 60  0001 C CNN
-F 3 "" H 9600 5050 60  0001 C CNN
-	1    9600 5050
+P 9700 5050
+F 0 "R21" V 9780 5050 50  0000 C CNN
+F 1 "1k" V 9700 5050 50  0000 C CNN
+F 2 "" H 9700 5050 60  0001 C CNN
+F 3 "" H 9700 5050 60  0001 C CNN
+	1    9700 5050
 	0    -1   -1   0
 $EndComp
@@
 	10350 5100 10350 5050
 Wire Wire Line
-	9000 5050 9350 5050
-Wire Wire Line
-	9300 5050 9300 5100
+	9000 5050 9550 5050
+Wire Wire Line
+	9300 5050 9300 5150
 $Comp
 L GND #PWR039
@@
 	10350 5550 10350 5500
 Wire Wire Line
-	9300 5500 9300 5550
+	9300 5450 9300 5550
 Connection ~ 9300 5050
 Connection ~ 10350 5050
@@
 L R R22
 U 1 1 50A1F50D
-P 9600 5750
-F 0 "R22" V 9680 5750 50  0000 C CNN
-F 1 "1k" V 9600 5750 50  0000 C CNN
-F 2 "" H 9600 5750 60  0001 C CNN
-F 3 "" H 9600 5750 60  0001 C CNN
-	1    9600 5750
+P 9700 5750
+F 0 "R22" V 9780 5750 50  0000 C CNN
+F 1 "1k" V 9700 5750 50  0000 C CNN
+F 2 "" H 9700 5750 60  0001 C CNN
+F 3 "" H 9700 5750 60  0001 C CNN
+	1    9700 5750
 	0    -1   -1   0
 $EndComp
@@
 	10350 5800 10350 5750
 Wire Wire Line
-	9000 5750 9350 5750
-Wire Wire Line
-	9300 5750 9300 5800
+	9000 5750 9550 5750
+Wire Wire Line
+	9300 5750 9300 5850
 $Comp
 L GND #PWR041
@@
 	10350 6250 10350 6200
 Wire Wire Line
-	9300 6200 9300 6250
+	9300 6150 9300 6250
 Connection ~ 9300 5750
 Connection ~ 10350 5750
@@
 	10300 5750 10700 5750
 $Comp
-L VCC #PWR?
+L VCC #PWR047
 U 1 1 50FE444D
 P 2550 1450
-F 0 "#PWR?" H 2550 1550 30  0001 C CNN
+F 0 "#PWR047" H 2550 1550 30  0001 C CNN
 F 1 "VCC" H 2550 1550 30  0000 C CNN
 F 2 "" H 2550 1450 60  0001 C CNN
@@
 Wire Wire Line
 	700  6550 700  1950
+$Comp
+L PWR_FLAG #FLG048
+U 1 1 58595ED5
+P 2450 1550
+F 0 "#FLG048" H 2450 1645 50  0001 C CNN
+F 1 "PWR_FLAG" H 2450 1730 50  0000 C CNN
+F 2 "" H 2450 1550 60  0000 C CNN
+F 3 "" H 2450 1550 60  0000 C CNN
+	1    2450 1550
+	1    0    0    -1
+$EndComp
+$Comp
+L PWR_FLAG #FLG049
+U 1 1 585962C3
+P 5450 3350
+F 0 "#FLG049" H 5450 3445 50  0001 C CNN
+F 1 "PWR_FLAG" H 5450 3530 50  0000 C CNN
+F 2 "" H 5450 3350 60  0000 C CNN
+F 3 "" H 5450 3350 60  0000 C CNN
+	1    5450 3350
+	-1   0    0    1
+$EndComp
+Wire Wire Line
+	5450 3350 5450 3250
+Wire Wire Line
+	5450 3250 5300 3250
+Connection ~ 5300 3250
+Wire Wire Line
+	1050 2250 1600 2250
+Wire Wire Line
+	1600 2150 1050 2150
 $EndSCHEMATC

Commit message: More connections and a net tie, ERC now passes
Parts:
- added NT101: Nettie, symbol Nettie
Connections:
- wire segments 236 -> 238
Changed lines of the file:
@@
 LIBS:contrib
 LIBS:valves
+LIBS:pyth
 LIBS:S88P-cache
 EELAYER 25 0
@@
 $EndComp
 Wire Wire Line
-	7750 1500 7750 1450
+	7750 1400 7750 1500
 Wire Wire Line
 	6900 1400 6900 1500
@@
 $EndComp
 Wire Wire Line
-	7750 2200 7750 2150
+	7750 2100 7750 2200
 Wire Wire Line
 	6900 2100 6900 2200
@@
 $EndComp
 Wire Wire Line
-	7750 2400 7750 2350
+	7750 2350 7750 2450
 Wire Wire Line
 	6600 2350 6950 2350
@@
 $EndComp
 Wire Wire Line
-	7750 2850 7750 2800
+	7750 2750 7750 2850
 Wire Wire Line
 	6900 2750 6900 2850
@@
 $EndComp
 Wire Wire Line
-	7750 3100 7750 3050
+	7750 3050 7750 3150
 Wire Wire Line
 	6600 3050 6950 3050
@@
 $EndComp
 Wire Wire Line
-	7750 3550 7750 3500
+	7750 3450 7750 3550
 Wire Wire Line
 	6900 3450 6900 3550
@@
 $EndComp
 Wire Wire Line
-	7750 3750 7750 3700
+	7750 3700 7750 3800
 Wire Wire Line
 	6600 3700 6950 3700
@@
 $EndComp
 Wire Wire Line
-	7750 4200 7750 4150
+	7750 4100 7750 4200
 Wire Wire Line
 	6900 4100 6900 4200
@@
 $EndComp
 Wire Wire Line
-	7750 4450 7750 4400
+	7750 4400 7750 4500
 Wire Wire Line
 	6600 4400 6950 4400
@@
 $EndComp
 Wire Wire Line
-	7750 4900 7750 4850
+	7750 4800 7750 4900
 Wire Wire Line
 	6900 4800 6900 4900
@@
 $EndComp
 Wire Wire Line
-	7750 5100 7750 5050
+	7750 5050 7750 5150
 Wire Wire Line
 	6600 5050 6950 5050
@@
 $EndComp
 Wire Wire Line
-	7750 5550 7750 5500
+	7750 5450 7750 5550
 Wire Wire Line
 	6900 5450 6900 5550
@@
 $EndComp
 Wire Wire Line
-	7750 5800 7750 5750
+	7750 5750 7750 5850
 Wire Wire Line
 	6600 5750 6950 5750
@@
 $EndComp
 Wire Wire Line
-	7750 6250 7750 6200
+	7750 6150 7750 6250
 Wire Wire Line
 	6900 6150 6900 6250
@@
 $EndComp
 Wire Wire Line
-	10350 1050 10350 1000
+	10350 1000 10350 1100
 Wire Wire Line
 	9000 1000 9550 1000
@@
 $EndComp
 Wire Wire Line
-	10350 1500 10350 1450
+	10350 1400 10350 1500
 Wire Wire Line
 	9300 1400 9300 1500
@@
 $EndComp
 Wire Wire Line
-	10350 1750 10350 1700
+	10350 1700 10350 1800
 Wire Wire Line
 	9000 1700 9550 1700
@@
 $EndComp
 Wire Wire Line
-	10350 2200 10350 2150
+	10350 2100 10350 2200
 Wire Wire Line
 	9300 2100 9300 2200
@@
 $EndComp
 Wire Wire Line
-	10350 2400 10350 2350
+	10350 2350 10350 2450
 Wire Wire Line
 	9000 2350 9550 2350
@@
 $EndComp
 Wire Wire Line
-	10350 2850 10350 2800
+	10350 2750 10350 2850
 Wire Wire Line
 	9300 2750 9300 2850
@@
 $EndComp
 Wire Wire Line
-	10350 3100 10350 3050
+	10350 3050 10350 3150
 Wire Wire Line
 	9000 3050 9550 3050
@@
 $EndComp
 Wire Wire Line
-	10350 3550 10350 3500
+	10350 3450 10350 3550
 Wire Wire Line
 	9300 3450 9300 3550
@@
 $EndComp
 Wire Wire Line
-	10350 3750 10350 3700
+	10350 3700 10350 3800
 Wire Wire Line
 	9000 3700 9550 3700
@@
 $EndComp
 Wire Wire Line
-	10350 4200 10350 4150
+	10350 4100 10350 4200
 Wire Wire Line
 	9300 4100 9300 4200
@@
 $EndComp
 Wire Wire Line
-	10350 4450 10350 4400
+	10350 4400 10350 4500
 Wire Wire Line
 	9000 4400 9550 4400
@@
 $EndComp
 Wire Wire Line
-	10350 4900 10350 4850
+	10350 4800 10350 4900
 Wire Wire Line
 	9300 4800 9300 4900
@@
 $EndComp
 Wire Wire Line
-	10350 5100 10350 5050
+	10350 5050 10350 5150
 Wire Wire Line
 	9000 5050 9550 5050
@@
 $EndComp
 Wire Wire Line
-	10350 5550 10350 5500
+	10350 5450 10350 5550
 Wire Wire Line
 	9300 5450 9300 5550
@@
 $EndComp
 Wire Wire Line
-	10350 5800 10350 5750
+	10350 5750 10350 5850
 Wire Wire Line
 	9000 5750 9550 5750
@@
 $EndComp
 Wire Wire Line
-	10350 6250 10350 6200
+	10350 6150 10350 6250
 Wire Wire Line
 	9300 6150 9300 6250
@@
 $EndComp
 Wire Wire Line
-	7250 1000 7300 1000
-Wire Wire Line
-	7700 1700 8050 1700
+	7250 1000 7350 1000
 Wire Bus Line
 	4800 750  8900 750
 Wire Wire Line
-	7700 1000 8100 1000
-Wire Wire Line
-	7750 1050 7750 1000
+	7650 1000 8100 1000
+Wire Wire Line
+	7750 1000 7750 1100
 Connection ~ 7750 1000
 $Comp
@@
 $EndComp
 Wire Wire Line
-	7250 5750 7300 5750
-Wire Wire Line
-	7700 5750 8100 5750
-Wire Wire Line
-	7700 5050 8050 5050
-Wire Wire Line
-	7300 5050 7250 5050
-Wire Wire Line
-	7250 4400 7300 4400
-Wire Wire Line
-	7700 4400 8000 4400
-Wire Wire Line
-	7250 3050 7300 3050
-Wire Wire Line
-	7700 3050 7950 3050
-Wire Wire Line
-	7700 3700 7950 3700
-Wire Wire Line
-	7300 3700 7250 3700
-Wire Wire Line
-	7250 1700 7300 1700
-Wire Wire Line
-	7250 2350 7300 2350
-Wire Wire Line
-	7700 2350 8000 2350
-Wire Wire Line
-	7750 1750 7750 1700
+	7250 5750 7350 5750
+Wire Wire Line
+	7650 5750 8100 5750
+Wire Wire Line
+	7650 5050 8050 5050
+Wire Wire Line
+	7250 5050 7350 5050
+Wire Wire Line
+	7250 4400 7350 4400
+Wire Wire Line
+	7650 4400 8000 4400
+Wire Wire Line
+	7250 3050 7350 3050
+Wire Wire Line
+	7650 3050 7950 3050
+Wire Wire Line
+	7650 3700 7950 3700
+Wire Wire Line
+	7250 3700 7350 3700
+Wire Wire Line
+	7250 1700 7350 1700
+Wire Wire Line
+	7250 2350 7350 2350
+Wire Wire Line
+	7650 2350 8000 2350
+Wire Wire Line
+	7750 1700 7750 1800
 Connection ~ 7750 1700
 $Comp
@@
 $EndComp
 Wire Wire Line
-	9850 1000 9900 1000
-Wire Wire Line
-	10300 1000 10700 1000
-Wire Wire Line
-	10300 1700 10650 1700
-Wire Wire Line
-	9900 1700 9850 1700
-Wire Wire Line
-	9850 2350 9900 2350
-Wire Wire Line
-	10300 2350 10600 2350
-Wire Wire Line
-	9850 3050 9900 3050
-Wire Wire Line
-	10300 3050 10550 3050
-Wire Wire Line
-	10300 3700 10550 3700
-Wire Wire Line
-	9900 3700 9850 3700
-Wire Wire Line
-	9850 4400 9900 4400
-Wire Wire Line
-	10300 4400 10600 4400
-Wire Wire Line
-	10300 5050 10650 5050
-Wire Wire Line
-	9900 5050 9850 5050
-Wire Wire Line
-	9850 5750 9900 5750
-Wire Wire Line
-	10300 5750 10700 5750
+	9850 1000 9950 1000
+Wire Wire Line
+	10250 1000 10700 1000
+Wire Wire Line
+	10250 1700 10650 1700
+Wire Wire Line
+	9850 1700 9950 1700
+Wire Wire Line
+	9850 2350 9950 2350
+Wire Wire Line
+	10250 2350 10600 2350
+Wire Wire Line
+	9850 3050 9950 3050
+Wire Wire Line
+	10250 3050 10550 3050
+Wire Wire Line
+	10250 3700 10550 3700
+Wire Wire Line
+	9850 3700 9950 3700
+Wire Wire Line
+	9850 4400 9950 4400
+Wire Wire Line
+	10250 4400 10600 4400
+Wire Wire Line
+	10250 5050 10650 5050
+Wire Wire Line
+	9850 5050 9950 5050
+Wire Wire Line
+	9850 5750 9950 5750
+Wire Wire Line
+	10250 5750 10700 5750
 $Comp
 L VCC #PWR047
@@
 Connection ~ 5300 3250
 Wire Wire Line
-	1050 2250 1600 2250
-Wire Wire Line
 	1600 2150 1050 2150
+$Comp
+L Nettie NT101
+U 1 1 58591D98
+P 1300 2250
+F 0 "NT101" H 1450 2200 60  0000 C CNN
+F 1 "Nettie" H 1300 2150 60  0000 C CNN
+F 2 "" H 1300 2250 60  0001 C CNN
+F 3 "" H 1300 2250 60  0001 C CNN
+	1    1300 2250
+	1    0    0    -1
+$EndComp
+Wire Wire Line
+	1050 2250 1150 2250
+Wire Wire Line
+	1450 2250 1600 2250
+Wire Wire Line
+	7700 2400 7750 2400
+Wire Wire Line
+	8050 1700 7650 1700
 $EndSCHEMATC
