File: Hardware/S88P3.kicad_pcb (KiCad board)
At the start: 2 copper layers, 59 x 40 mm, 84 parts, among them IC1 ATMEGA8-AI, J1 RJ45, J2 RJ45, P1 CONN_3X2, P2 CONN_8, P3 CONN_8

Commit message: Finished component modernisation
Parts:
- added NT101: Nettie, Other:nettie_0.3mm, B.Cu at (134.8, 183.6)
- C1, C10, C11, C12, C13, C14, C15, C16, C17, C18, C2, C3, C4, C5, C6, C7, C8, C9, D18, D19, D20, D21, D22, D23, D24, D25, D26, D27, D28, D29, D30, D31, D32, D33: footprint SM0805 -> Capacitors_SMD:C_0805
- D1: footprint LED-0805 -> LEDs:LED-0805
- D10, D11, D12, D13, D14, D15, D16, D17, D2, D3, D4, D5, D6, D7, D8, D9: footprint D3 -> Discret:D3
- IC1: footprint TQFP32 -> Housings_QFP:TQFP-32_7x7mm_Pitch0.8mm
- J1, J2: footprint RJ45_8 -> Connect:RJ45_8
- P1: footprint pin_array_3x2 -> Socket_Strips:Socket_Strip_Straight_2x03; moved to B.Cu
- P2, P3: footprint 9PIN_SC_RM3.5 -> screw_connector:9PIN_SC_RM3.5
- R1, R10, R11, R12, R13, R14, R15, R16, R17, R18, R19, R2, R20, R21, R22, R3, R4, R5, R6, R7, R8, R9: footprint SM0805 -> Resistors_SMD:R_0805
- moved P1 2.69 mm to (150.9, 166.6)
- moved C16 0.23 mm to (119.5, 183.2)
- moved D31 0.23 mm to (119.5, 187.2)
- moved R20 0.23 mm to (119.5, 185.2)
- turned D10 to 180 degrees
- turned D11 to 180 degrees
- turned D12 to 180 degrees
- turned D13 to 180 degrees
- turned D14 to 180 degrees
- turned D15 to 180 degrees
- turned D16 to 180 degrees
- turned D17 to 180 degrees
- turned D2 to 0 degrees
- turned D3 to 0 degrees
- turned D4 to 0 degrees
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Routing:
- net Net-(D14-Pad2): track 11.3 -> 15.6 mm
- net Net-(D16-Pad2): track 16.4 -> 15.5 mm
- net VCC: track 105.6 -> 104.8 mm
